File: KiCad/DeFocuserLiteSMD.kicad_sch (KiCad schematic)
At the start: 22 parts, among them M1 MTR, U1 MOUDLE-SEEEDUINO-XIAO-ESP32C3, U2 MT3608, U3 TMC2209-LA-T

Commit message: Part number update
Parts:
- C4: LCSC Part C2170367 -> C2180991
Changed lines of the file:
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@@
 			)
 		)
-		(property "LCSC Part" "C2170367"
+		(property "LCSC Part" "C2180991"
 			(at 219.71 143.51 0)
 			(effects

Commit message: Fixed resistor value + reexported BOM
Parts:
- R3: LCSC Part C5138992 -> C137099
- R4: LCSC Part (none) -> C137099
Changed lines of the file:
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@@
+			)
+		)
+		(property "LCSC Part" "C137099"
+			(at 220.98 109.22 90)
+			(effects
+				(font
+					(size 1.27 1.27)
+				)
+				(hide yes)
 			)
 		)
@@
 			)
 		)
-		(property "LCSC Part" "C5138992"
+		(property "LCSC Part" "C137099"
 			(at 220.98 119.38 90)
 			(effects

Commit message: Added lcsc part numbers with in stock components
Parts:
- C1, C2: LCSC Part (none) -> C5348165
- D1: LCSC Part (none) -> C908680
- L1: LCSC Part (none) -> C87002
- R1: LCSC Part (none) -> C2933708
- R2: LCSC Part (none) -> C2907446
- R5: LCSC Part (none) -> C17902
- R6: LCSC Part (none) -> C2907440
- S1: LCSC Part (none) -> C720477
- U2: LCSC Part (none) -> C84817
Changed lines of the file:
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@@
+			)
+		)
+		(property "LCSC Part" "C720477"
+			(at 125.73 81.28 0)
+			(effects
+				(font
+					(size 1.27 1.27)
+				)
+				(hide yes)
 			)
 		)
@@
 			)
 		)
+		(property "LCSC Part" "C5348165"
+			(at 160.02 63.5 0)
+			(effects
+				(font
+					(size 1.27 1.27)
+				)
+				(hide yes)
+			)
+		)
 		(pin "2"
 		)
@@
 			)
 		)
+		(property "LCSC Part" "C84817"
+			(at 173.99 59.69 0)
+			(effects
+				(font
+					(size 1.27 1.27)
+				)
+				(hide yes)
+			)
+		)
 		(pin "5"
 		)
@@
 			)
 		)
+		(property "LCSC Part" "C2907446"
+			(at 195.58 68.58 0)
+			(effects
+				(font
+					(size 1.27 1.27)
+				)
+				(hide yes)
+			)
+		)
 		(pin "2"
 		)
@@
 			)
 		)
+		(property "LCSC Part" "C87002"
+			(at 173.99 45.72 0)
+			(effects
+				(font
+					(size 1.27 1.27)
+				)
+				(hide yes)
+			)
+		)
 		(pin "2"
 		)
@@
 			)
 		)
+		(property "LCSC Part" "C2907440"
+			(at 161.29 133.35 90)
+			(effects
+				(font
+					(size 1.27 1.27)
+				)
+				(hide yes)
+			)
+		)
 		(pin "1"
 		)
@@
 		)
 		(property "Description" "Resistor"
+			(at 118.11 88.9 0)
+			(effects
+				(font
+					(size 1.27 1.27)
+				)
+				(hide yes)
+			)
+		)
+		(property "LCSC Part" "C17902"
 			(at 118.11 88.9 0)
 			(effects
@@
 			)
 		)
+		(property "LCSC Part" "C5348165"
+			(at 207.01 53.34 0)
+			(effects
+				(font
+					(size 1.27 1.27)
+				)
+				(hide yes)
+			)
+		)
 		(pin "2"
 		)
@@
 			)
 		)
+		(property "LCSC Part" "C2933708"
+			(at 195.58 52.07 0)
+			(effects
+				(font
+					(size 1.27 1.27)
+				)
+				(hide yes)
+			)
+		)
 		(pin "2"
 		)
@@
 			(at 189.23 45.72 0)
 			(effects
+				(font
+					(size 1.27 1.27)
+				)
+				(hide yes)
+			)
+		)
+		(property "LCSC Part" "C908680"
+			(at 189.23 45.72 0)
+			(effects

Commit message: Trying V2 with better pcb layout to expose I2C, and new driver with standalone app integrated as a mediator
Parts:
- added JP1: SolderJumper_3_Open, Jumper:SolderJumper-3_P1.3mm_Open_RoundedPad1.0x1.5mm_NumberLabels, symbol Jumper:SolderJumper_3_Open
- added M2: MTR, Connector_JST:JST_XH_B4B-XH-A_1x04_P2.50mm_Vertical, symbol Connector_Generic:Conn_01x04
Connections:
- net +5V: now also JP1.1 (A)
- net DIAG: now also U1.1 (PA02_A0_D0); no longer U1.3 (PA10_A2_D2)
- net DIR: now also U1.3 (PA10_A2_D2); no longer U1.6 (PA9_A5_D5_SCL)
- net GND: now also M2.4 (Pin_4)
- net STP: now also U1.2 (PA4_A1_D1); no longer U1.5 (PA8_A4_D4_SDA)
- net +3.3V: now reaches U1.12 (3V3)
- net +3.3V: now also JP1.3 (B)
- new net: JP1.2 (C), M2.1 (Pin_1)
- new net SCL: M2.3 (Pin_3), U1.6 (PA9_A5_D5_SCL)
- new net SDA: M2.2 (Pin_2), U1.5 (PA8_A4_D4_SDA)
- no-connect marks 8 -> 7
